File: BIG_MUFF.kicad_pcb (KiCad board)
At the start: 2 copper layers, 55 x 71 mm, 58 parts, among them J1 9V DC, J2 IN, J3 OUT, J4 PINHD_1x3_Female, J5 PINHD_1x3_Male, Q1 BC547, Q2 BC547, Q3 BC547, Q4 BC547, SW6 SW_3PDT_Footswitch

Commit message: DRM fix
Parts:
- added G***: LOGO, LOGO, F.Cu at (161.8, 133.8)
- added H1: ~, PCM_fab:MountingHole_M2, F.Cu at (174.2, 83.2)
- added H2: ~, PCM_fab:MountingHole_M2, F.Cu at (142.5, 83.0)
- added H3: ~, PCM_fab:MountingHole_M2, F.Cu at (175.2, 125.5)
- moved D4 3.01 mm to (160.8, 68.2)
- moved R11 2.90 mm to (158.0, 72.0)
- moved R25 2.50 mm to (139.5, 72.7)
- moved R20 2.44 mm to (142.0, 72.8)
- moved J5 1.16 mm to (176.1, 136.0)
- moved D1 0.59 mm to (140.5, 95.3)
- moved R1 0.53 mm to (172.5, 122.5)
Routing:
- net /Q3_C: track 51.9 -> 56.2 mm
- net /TONE_LO: track 19.8 -> 22.4 mm
- net /TONE_IN: track 55.2 -> 57.7 mm
- net /Q1_B: track 42.0 -> 44.5 mm
- net /Q3_B: track 32.2 -> 34.6 mm
- net Net-(F1-Pad1): track 3.67 -> 5.38 mm
- net /OUTPUT: track 43.6 -> 45.2 mm
- net /+9V: track 144.7 -> 146.3 mm
- net /TONE_HI: track 52.3 -> 53.7 mm
- net /Q4_B: track 20.5 -> 21.1 mm
- net /+DC_PWR: track 4.95 -> 5.45 mm
Other:
- board text added: "/ C0DE-Z"

Commit message: prod ready for jcl
Parts:
- added G***: LOGO, LOGO, B.Cu at (167.5, 107.7)
- moved G*** 1.27 mm to (160.5, 133.5)
- moved C9 0.75 mm to (140.5, 127.0)
- moved SW6 0.55 mm to (145.8, 124.3)
- moved D4 0.50 mm to (161.2, 68.2)
- moved R11 0.50 mm to (158.5, 72.0)
- moved R20 0.50 mm to (142.5, 72.8)
- moved R23 0.50 mm to (148.0, 80.0)
- moved R25 0.50 mm to (140.0, 72.7)
- moved R26 0.50 mm to (129.5, 80.0)
- moved R5 0.50 mm to (166.5, 80.0)
Routing:
- net /TIP: track 56.5 -> 70.6 mm
- net /Q2_C: track 32.0 -> 35.7 mm
- net /+9V: track 146.3 -> 143.5 mm
- net /TONE_IN: track 57.7 -> 60.5 mm
- net /TONE_LO: track 22.4 -> 23.4 mm
- net /Q3_B: track 34.6 -> 35.4 mm
- net /Q3_C: track 56.2 -> 55.5 mm

Commit message: ready for jcl
Parts:
- added ?: , , F.Cu at (125.5, 78.5)
Other:
- board text added: "Let's All Walk Each Other Home"

Commit message: fix routing
Parts:
- moved ? 0.50 mm to (125.0, 78.5)
Routing:
- net /TONE_HI: track 53.7 -> 54.4 mm
Other:
- board text added: "ECSTATIS"
- board text added: "Mk2"
- board text removed: "Mk1"
