File: _restore_backup_2026-10-06T00-20-56-311/BIG_MUFF.kicad_pcb (KiCad board)
At the start: 2 copper layers, 55 x 71 mm, 64 parts, among them J1 9V DC, J2 IN, J3 OUT, J4 PINHD_1x3_Female, J5 PINHD_1x3_Male, Q1 BC547, Q2 BC547, Q3 BC547, Q4 BC547, SW6 SW_3PDT_Footswitch

Commit message: mk2
Routing:
- net /+9V: track 141.8 -> 144.7 mm, vias 1 -> 7
- net /CATHODE: track 41.8 -> 41.0 mm
- net /Q3_C: track 55.7 -> 55.5 mm, vias 2 -> 3
Other:
- board text removed: "9V IN"
- board text removed: "DIST"
- board text removed: "IN"
- board text removed: "OUT"
- board text removed: "TONE"
- board text removed: "VOLUME"
